Commit message: Its walking!

File: assets/mini_cheetah.urdf (robot description, URDF)
Before this commit: robot mini_cheetah_vision, 18 links, 17 joints
Links:
- link FL_calf: geometry collision box size=0.025 0.025 0.1955; visual mesh filename=meshes/lower_leg.dae
- link FL_hip: geometry visual mesh filename=meshes/mini_vision_abd.dae
- link FL_thigh: geometry collision box size=0.2585 0.034 0.043; visual mesh filename=meshes/mini_vision_shank.dae
- link FR_calf: geometry collision box size=0.025 0.025 0.1955; visual mesh filename=meshes/lower_leg.dae
- link FR_hip: geometry visual mesh filename=meshes/mini_vision_abd.dae
- link FR_thigh: geometry collision box size=0.2585 0.034 0.043; visual mesh filename=meshes/mini_vision_shank.dae
- link RL_calf: geometry collision box size=0.025 0.025 0.1955; visual mesh filename=meshes/lower_leg.dae
- link RL_hip: geometry visual mesh filename=meshes/mini_vision_abd.dae
- link RL_thigh: geometry collision box size=0.2585 0.034 0.043; visual mesh filename=meshes/mini_vision_shank.dae
- link RR_calf: geometry collision box size=0.025 0.025 0.1955; visual mesh filename=meshes/lower_leg.dae
- link RR_hip: geometry visual mesh filename=meshes/mini_vision_abd.dae
- link RR_thigh: geometry collision box size=0.2585 0.034 0.043; visual mesh filename=meshes/mini_vision_shank.dae
- link trunk: geometry collision mesh filename=meshes/mini_vision_body.dae scale=1 1 1; visual mesh filename=meshes/mini_vision_body.dae scale=1 1 1
